Commit message: Fix parol6 URDF kinematics: replace with the parol6 pip package's own URDF
The ros_parol/src/parol6/urdf/parol6.urdf shipped in this repo (a
SolidWorks-exported URDF) does not match the kinematics of PAROL6_ROBOT.py
in the PAROL6-python-API pip package (parol6/urdf_model/urdf/PAROL6.urdf),
which is the URDF actually used for parol6-server's own forward
kinematics, joint limits, and collision checking.

The mismatch is not a small numeric drift -- several joints (L3, L4, L5,
L6) have opposite rotation axis signs (0 0 1 vs 0 0 -1) between the two
files, and the joint limit ranges for L2 and L3 barely overlap at all
(e.g. L3: [-2, 1.3] rad in this repo's URDF vs [1.88, 5.02] rad in
PAROL6_ROBOT.py's -- the two ranges don't even share a value near zero).
Driving ros2_control from this repo's URDF against a real/simulated
parol6-server means joint-limit checks reject valid poses (observed: the
robot's actual home position is invalid per this URDF's stated L3 limit)
and, more importantly, forward kinematics disagree with the robot's own
kinematic model -- so any pose reasoning done against this URDF (IK
seeding, collision checking, Cartesian planning) does not correspond to
where the physical arm actually is.

Fix: replace this URDF with the one already shipped in and used by the
PAROL6-python-API pip package, so there is exactly one authoritative
kinematic description instead of two independently-exported ones drifting
apart. Also add the *_simplified.stl collision meshes it references,
which existed in the pip package's mesh set but not here.

Verified by forward-kinematics comparison: for a test configuration
(q = [10, -30, 150, 20, -10, 30] degrees), PAROL6_ROBOT.py's
robot.fkine(q) and this repo's URDF (loaded via robot_state_publisher,
queried via `ros2 run tf2_ros tf2_echo`) now produce matching transforms
to displayed precision. Before this fix they did not agree at all (not
just numerically off -- effectively unrelated poses).

Tested via ros2_control (not this repo's MoveIt config, which wasn't
available on the ROS2 distro used for testing) against a real
parol6-server instance, with a real PAROL6SystemInterface plugin
(https://github.com/grahas/parol6_ros2_control) driving the hardware
side, using the server's own software simulator mode (no physical robot
motion involved in verification).

Co-Authored-By: Claude Sonnet 5 <noreply@anthropic.com>

File: ros_parol/src/parol6/urdf/parol6.urdf (robot description, URDF)
Before this commit: robot parol6, 8 links, 7 joints
Links:
- link L1: geometry collision mesh filename=package://parol6/meshes/L1_simplified.stl; visual mesh filename=package://parol6/meshes/L1.STL
- link L2: geometry collision mesh filename=package://parol6/meshes/L2_simplified.stl; visual mesh filename=package://parol6/meshes/L2.STL
- link L3: geometry collision mesh filename=package://parol6/meshes/L3_simplified.stl; visual mesh filename=package://parol6/meshes/L3.STL
- link L4: geometry collision mesh filename=package://parol6/meshes/L4_simplified.stl; visual mesh filename=package://parol6/meshes/L4.STL
- link L5: geometry collision mesh filename=package://parol6/meshes/L5_simplified.stl; visual mesh filename=package://parol6/meshes/L5.STL
- link L6: geometry collision mesh filename=package://parol6/meshes/L6_simplified.stl; visual mesh filename=package://parol6/meshes/L6.STL
- link base_link: geometry collision mesh filename=package://parol6/meshes/base_link_simplified.stl; visual mesh filename=package://parol6/meshes/base_link.STL
Joints:
- joint L1: limit lower=-1.7 upper=1.7 effort=300 velocity=3 -> lower=-2.1475731 upper=2.1475731 effort=300 velocity=3; origin xyz=0 0 0 rpy=0 0 0 -> xyz=0 0 0.1105 rpy=0 0 0
- joint L2: limit lower=-0.98 upper=1 effort=300 velocity=3 -> lower=-2.530881 upper=-0.05890486 effort=300 velocity=3; origin xyz=0.0234207210610375 0 0.1105 rpy=-1.5707963267949 0 0 -> xyz=0.0234207210610375 0 0 rpy=-1.5707963267949 0 0
- joint L3: axis 0 0 -1 -> 0 0 1; limit lower=-2 upper=1.3 effort=300 velocity=3 -> lower=1.88261685 upper=5.02423568 effort=300 velocity=3; origin xyz=0 -0.18 0 rpy=3.1416 0 -1.5708 -> xyz=0.18 0 0 rpy=3.14159265358979 0 0
- joint L4: axis 0 0 -1 -> 0 0 1; limit lower=-2 upper=2 effort=300 velocity=3 -> lower=-1.8407944 upper=1.8407944 effort=300 velocity=3; origin xyz=0.0435 0 0 rpy=1.5707963267949 0 3.14159265358979 -> xyz=-0.0435 0.17635 0 rpy=1.5707963267949 0 0
- joint L5: axis 0 0 -1 -> 0 0 1; limit lower=-2.1 upper=2.1 effort=300 velocity=3 -> lower=-1.57079633 upper=1.57079633 effort=300 velocity=3; origin xyz=0 0 -0.17635 rpy=-1.5708 0 0 -> xyz=0 0 0 rpy=-1.5707963267949 0 0
- joint L6: axis 0 0 -1 -> 0 0 1; limit lower=-3.1 upper=3.1 effort=300 velocity=3 -> lower=0.0 upper=6.28318531 effort=300 velocity=3; origin xyz=0 0 0 rpy=1.5708 0 0 -> xyz=0 0.037 0 rpy=1.5707963267949 0 0; type continuous -> revolute
