Commit message: Fix tool jaw TF errors and mesh orientation
Jaw joints (tool_left_jaw_joint/tool_right_jaw_joint) were declared
prismatic, but nothing publishes /joint_states for them since they are
not ros2_control-actuated (grippers are driven via parol6's own
tool_action()/select_tool() API). A non-fixed joint needs a live state
value to resolve its transform at all, so robot_state_publisher could
not compute these transforms, producing "No transform from
tool_left_jaw to world" TF errors and undefined rendering in RViz.
Changed to fixed joints across pneumatic, ssg48, and msg grippers.

Also removed an incorrect Rx(pi) rotation applied to every tool body
and jaw mesh's visual/collision origin. Checking each mesh's own
bounding box against its tools.py tcp_xyz shows the meshes are already
authored directly in the flange/L6 frame, extending toward -Z to match
the (negative) tcp_xyz values; the added Rx(pi) instead flipped the
tool to point back into the wrist, visually colliding with the robot
body. Removed for pneumatic, ssg48, msg, and vacuum.

File: ros_parol/src/parol6/urdf/tools/msg_gripper.xacro (robot description, xacro)
@@ -33,9 +33,9 @@
     <link name="tool_body">
       <visual>
-        <origin xyz="0 0 0" rpy="${pi} 0 0" />
+        <origin xyz="0 0 0" rpy="0 0 0" />
         <geometry><mesh filename="${mesh_body}" /></geometry>
       </visual>
       <collision>
-        <origin xyz="0 0 0" rpy="${pi} 0 0" />
+        <origin xyz="0 0 0" rpy="0 0 0" />
         <geometry><mesh filename="${mesh_body}" /></geometry>
       </collision>
@@ -48,35 +48,37 @@
     <link name="tool_right_jaw">
       <visual>
-        <origin xyz="0 0 0" rpy="${pi} 0 0" />
+        <origin xyz="0 0 0" rpy="0 0 0" />
         <geometry><mesh filename="${mesh_right_jaw}" /></geometry>
       </visual>
       <collision>
-        <origin xyz="0 0 0" rpy="${pi} 0 0" />
+        <origin xyz="0 0 0" rpy="0 0 0" />
         <geometry><mesh filename="${mesh_right_jaw}" /></geometry>
       </collision>
     </link>
-    <joint name="tool_right_jaw_joint" type="prismatic">
+    <!-- Fixed, not prismatic: a movable joint here would need a live
+         position from /joint_states to resolve its transform at all,
+         and nothing publishes one for these (not ros2_control-actuated,
+         see file header), resulting in "No transform" TF errors rather
+         than just a static, non-animated pose. See pneumatic_gripper.xacro
+         for the fuller explanation. -->
+    <joint name="tool_right_jaw_joint" type="fixed">
       <parent link="${parent}" />
       <child link="tool_right_jaw" />
       <origin xyz="0 0 0" rpy="0 0 0" />
-      <axis xyz="${jaw_axis_x} ${jaw_axis_y} ${jaw_axis_z}" />
-      <limit lower="0" upper="${jaw_travel}" effort="20" velocity="0.1" />
     </joint>
     <link name="tool_left_jaw">
       <visual>
-        <origin xyz="0 0 0" rpy="${pi} 0 0" />
+        <origin xyz="0 0 0" rpy="0 0 0" />
         <geometry><mesh filename="${mesh_left_jaw}" /></geometry>
       </visual>
       <collision>
-        <origin xyz="0 0 0" rpy="${pi} 0 0" />
+        <origin xyz="0 0 0" rpy="0 0 0" />
         <geometry><mesh filename="${mesh_left_jaw}" /></geometry>
       </collision>
     </link>
-    <joint name="tool_left_jaw_joint" type="prismatic">
+    <joint name="tool_left_jaw_joint" type="fixed">
       <parent link="${parent}" />
       <child link="tool_left_jaw" />
       <origin xyz="0 0 0" rpy="0 0 0" />
-      <axis xyz="${-jaw_axis_x} ${-jaw_axis_y} ${-jaw_axis_z}" />
-      <limit lower="0" upper="${jaw_travel}" effort="20" velocity="0.1" />
     </joint>
     <link name="tool_tcp" />

File: ros_parol/src/parol6/urdf/tools/pneumatic_gripper.xacro (robot description, xacro)
@@ -42,15 +42,16 @@
       <xacro:property name="tcp_xyz" value="0.0 0.0 -0.082" />
     </xacro:unless>
-    <!-- Body: fixed to the flange. All parol6 tool meshes are authored with
-         an Rx(pi) convention relative to the flange/kinematic frame. The
-         kinematic chain (TCP transform, jaw axes) stays pure translation,
-         and the rotation is applied only to mesh visuals/collisions. -->
+    <!-- Body: fixed to the flange, no rotation. All parol6 tool meshes are
+         authored directly in the flange/L6 frame (mounting face at the
+         mesh origin, body/jaws extending toward -Z, matching tcp_xyz's
+         negative Z below), confirmed by checking each mesh's own
+         bounding box against its tools.py tcp_xyz. -->
     <link name="tool_body">
       <visual>
-        <origin xyz="0 0 0" rpy="${pi} 0 0" />
+        <origin xyz="0 0 0" rpy="0 0 0" />
         <geometry><mesh filename="${mesh_body}" /></geometry>
       </visual>
       <collision>
-        <origin xyz="0 0 0" rpy="${pi} 0 0" />
+        <origin xyz="0 0 0" rpy="0 0 0" />
         <geometry><mesh filename="${mesh_body}" /></geometry>
       </collision>
@@ -61,39 +62,46 @@
       <origin xyz="0 0 0" rpy="0 0 0" />
     </joint>
-    <!-- Jaws: prismatic, symmetric (move in opposite directions along the
-         same axis). Not ros2_control-actuated, see file header. -->
+    <!-- Jaws: fixed at their as-modeled mesh position (jaw_axis/jaw_travel
+         above describe the real linear travel for documentation, but
+         aren't applied to a movable joint here). These would need to be
+         prismatic to actually animate open/closed, but a prismatic (or
+         any non-fixed) joint requires a live position from /joint_states
+         to resolve its transform at all, and since these joints aren't
+         ros2_control-actuated (see file header) and nothing else
+         publishes a state for them, robot_state_publisher can't compute
+         their transform, and TF/RViz shows them as unresolved ("No
+         transform from tool_left_jaw to world") rather than just static.
+         Fixed avoids that entirely; animating the jaws for real would
+         need a small joint_state_publisher-style node driven by
+         RobotClient.tool.status().positions, not attempted here. -->
     <link name="tool_right_jaw">
       <visual>
-        <origin xyz="0 0 0" rpy="${pi} 0 0" />
+        <origin xyz="0 0 0" rpy="0 0 0" />
         <geometry><mesh filename="${mesh_right_jaw}" /></geometry>
       </visual>
       <collision>
-        <origin xyz="0 0 0" rpy="${pi} 0 0" />
+        <origin xyz="0 0 0" rpy="0 0 0" />
         <geometry><mesh filename="${mesh_right_jaw}" /></geometry>
       </collision>
     </link>
-    <joint name="tool_right_jaw_joint" type="prismatic">
+    <joint name="tool_right_jaw_joint" type="fixed">
       <parent link="${parent}" />
       <child link="tool_right_jaw" />
       <origin xyz="0 0 0" rpy="0 0 0" />
-      <axis xyz="${jaw_axis_x} ${jaw_axis_y} ${jaw_axis_z}" />
-      <limit lower="0" upper="${jaw_travel}" effort="20" velocity="0.1" />
     </joint>
     <link name="tool_left_jaw">
       <visual>
-        <origin xyz="0 0 0" rpy="${pi} 0 0" />
+        <origin xyz="0 0 0" rpy="0 0 0" />
         <geometry><mesh filename="${mesh_left_jaw}" /></geometry>
       </visual>
       <collision>
-        <origin xyz="0 0 0" rpy="${pi} 0 0" />
+        <origin xyz="0 0 0" rpy="0 0 0" />
         <geometry><mesh filename="${mesh_left_jaw}" /></geometry>
       </collision>
     </link>
-    <joint name="tool_left_jaw_joint" type="prismatic">
+    <joint name="tool_left_jaw_joint" type="fixed">
       <parent link="${parent}" />
       <child link="tool_left_jaw" />
       <origin xyz="0 0 0" rpy="0 0 0" />
-      <axis xyz="${-jaw_axis_x} ${-jaw_axis_y} ${-jaw_axis_z}" />
-      <limit lower="0" upper="${jaw_travel}" effort="20" velocity="0.1" />
     </joint>
     <!-- TCP: pure translation from the flange, matching parol6-server's

File: ros_parol/src/parol6/urdf/tools/ssg48_gripper.xacro (robot description, xacro)
@@ -22,9 +22,9 @@
     <link name="tool_body">
       <visual>
-        <origin xyz="0 0 0" rpy="${pi} 0 0" />
+        <origin xyz="0 0 0" rpy="0 0 0" />
         <geometry><mesh filename="${mesh_body}" /></geometry>
       </visual>
       <collision>
-        <origin xyz="0 0 0" rpy="${pi} 0 0" />
+        <origin xyz="0 0 0" rpy="0 0 0" />
         <geometry><mesh filename="${mesh_body}" /></geometry>
       </collision>
@@ -37,35 +37,37 @@
     <link name="tool_right_jaw">
       <visual>
-        <origin xyz="0 0 0" rpy="${pi} 0 0" />
+        <origin xyz="0 0 0" rpy="0 0 0" />
         <geometry><mesh filename="${mesh_right_jaw}" /></geometry>
       </visual>
       <collision>
-        <origin xyz="0 0 0" rpy="${pi} 0 0" />
+        <origin xyz="0 0 0" rpy="0 0 0" />
         <geometry><mesh filename="${mesh_right_jaw}" /></geometry>
       </collision>
     </link>
-    <joint name="tool_right_jaw_joint" type="prismatic">
+    <!-- Fixed, not prismatic: a movable joint here would need a live
+         position from /joint_states to resolve its transform at all,
+         and nothing publishes one for these (not ros2_control-actuated,
+         see file header), resulting in "No transform" TF errors rather
+         than just a static, non-animated pose. See pneumatic_gripper.xacro
+         for the fuller explanation. -->
+    <joint name="tool_right_jaw_joint" type="fixed">
       <parent link="${parent}" />
       <child link="tool_right_jaw" />
       <origin xyz="0 0 0" rpy="0 0 0" />
-      <axis xyz="${jaw_axis_x} ${jaw_axis_y} ${jaw_axis_z}" />
-      <limit lower="0" upper="${jaw_travel}" effort="20" velocity="0.1" />
     </joint>
     <link name="tool_left_jaw">
       <visual>
-        <origin xyz="0 0 0" rpy="${pi} 0 0" />
+        <origin xyz="0 0 0" rpy="0 0 0" />
         <geometry><mesh filename="${mesh_left_jaw}" /></geometry>
       </visual>
       <collision>
-        <origin xyz="0 0 0" rpy="${pi} 0 0" />
+        <origin xyz="0 0 0" rpy="0 0 0" />
         <geometry><mesh filename="${mesh_left_jaw}" /></geometry>
       </collision>
     </link>
-    <joint name="tool_left_jaw_joint" type="prismatic">
+    <joint name="tool_left_jaw_joint" type="fixed">
       <parent link="${parent}" />
       <child link="tool_left_jaw" />
       <origin xyz="0 0 0" rpy="0 0 0" />
-      <axis xyz="${-jaw_axis_x} ${-jaw_axis_y} ${-jaw_axis_z}" />
-      <limit lower="0" upper="${jaw_travel}" effort="20" velocity="0.1" />
     </joint>
     <link name="tool_tcp" />

File: ros_parol/src/parol6/urdf/tools/vacuum_gripper.xacro (robot description, xacro)
@@ -14,9 +14,9 @@
     <link name="tool_body">
       <visual>
-        <origin xyz="0 0 0" rpy="${pi} 0 0" />
+        <origin xyz="0 0 0" rpy="0 0 0" />
         <geometry><mesh filename="package://parol6/meshes/vacuum_gripper_body_simplified.stl" /></geometry>
       </visual>
       <collision>
-        <origin xyz="0 0 0" rpy="${pi} 0 0" />
+        <origin xyz="0 0 0" rpy="0 0 0" />
         <geometry><mesh filename="package://parol6/meshes/vacuum_gripper_body_simplified.stl" /></geometry>
       </collision>

Commit message: Fix MSG gripper body mount offset
Unlike the pneumatic/ssg48/vacuum bodies, whose mount face sits exactly
flush at z=0 in the flange frame, the MSG body mesh's mount face is at
z=+0.0065, poking 6.5mm past the flange face into the wrist's own mesh
volume. Confirmed by live testing on real hardware across all three
rail-length variants (100/150/200mm, which share the same body mesh):
the gripper body visibly overlapped the wrist in RViz.

Shifted tool_body_joint back by 0.0065m to bring the mount face flush
with z=0, matching the other tool bodies' convention. Jaws are
untouched since they don't protrude past z=0. Some residual visual
closeness to the wrist remains after this fix and is expected: the
MSG body's mounting-block footprint (~6.7cm x 5.4cm) is inherently
wider than the flange (L6, ~3.2cm x 3.2cm), so any overlap in Z near
the mount will visually wrap around the flange's sides.

File: ros_parol/src/parol6/urdf/tools/msg_gripper.xacro (robot description, xacro)
@@ -31,4 +31,9 @@
       <xacro:property name="jaw_travel" value="0.0767" />
     </xacro:if>
+    <!-- Unlike the other tool bodies (pneumatic/ssg48/vacuum), this mesh's
+         mount face isn't flush at z=0, it extends to z=+0.0065, poking
+         past the flange face into the wrist's own mesh volume. Shifted
+         back by that amount so the mount face lands at z=0 like the
+         others; jaws are untouched since they don't protrude past z=0. -->
     <link name="tool_body">
       <visual>
@@ -44,5 +49,5 @@
       <parent link="${parent}" />
       <child link="tool_body" />
-      <origin xyz="0 0 0" rpy="0 0 0" />
+      <origin xyz="0 0 -0.0065" rpy="0 0 0" />
     </joint>
     <link name="tool_right_jaw">
