Commit message: Add ros2_control integration: hardware interface, bridge, bringup
Adds three new packages (mirrored from github.com/grahas/parol6_ros2_control,
kept in sync there as the primary development repo):

- parol6_hardware_interface: a hardware_interface::SystemInterface plugin
  (Parol6SystemInterface) driving the real robot via streaming servo_j()
  through a local TCP bridge. Targets the newer ros2_control
  HardwareComponentInterfaceParams-based API generation, not Humble's --
  builds against ROS2 "lyrical" (verified), not this repo's Humble-based
  demo.launch.py/mock hardware path.
- parol6_bridge: the TCP<->UDP daemon between the C++ plugin and
  parol6-server, reusing the parol6 Python SDK's wire protocol directly
  rather than reimplementing it in C++.
- parol6_bringup: a standalone bringup (launch + controllers.yaml) for
  driving the arm via ros2_control without MoveIt, used and validated
  independently of parol6_moveit.

parol6_moveit changes, layered on top of the tool support in this branch:
- config/parol6.urdf.xacro, config/parol6.srdf: plan against "tool_tcp"
  (the mounted tool's actual working point) instead of the bare flange
  L6, plus disable_collisions entries for the pneumatic gripper's
  body/jaw links against L5/L6 (needed once tool_tcp is in the group --
  their fixed-joint mount was otherwise flagged as a self-collision).
- config/initial_positions.yaml: was all-zero, which is invalid -- L2's
  URDF joint limit is [-2.5309, -0.0589] rad and L3's is
  [1.8826, 5.0242] rad, neither including zero. Found by actually
  running MoveIt planning against this config for the first time ever
  ("Motion planning start tree could not be initialized!"). Replaced
  with parol6's own real HOME_ANGLES_DEG (parol6/config.py).
- config/moveit_controllers.yaml: was missing action_ns entirely, so
  moveit_simple_controller_manager couldn't find the controller's
  FollowJointTrajectory action server ("Unable to identify any set of
  controllers that can actuate the specified joints"), even though the
  controller was running and correctly named. Also renamed the
  controller from arm_group_controller to parol6_arm_controller to
  match parol6_bringup's, so both packages drive the same controller
  name.
- config/parol6.ros2_control.xacro, launch/real_robot.launch.py,
  package.xml: use_real_hardware toggle -- swaps mock_components for
  Parol6SystemInterface, starts parol6_bridge, and lets MoveIt plan
  against the real bridge/parol6-server instead of only mock hardware.

Verified: parol6/parol6_bridge/parol6_bringup/parol6_moveit build clean
under ROS2 Humble; parol6_hardware_interface builds clean under ROS2
lyrical (its actual target). A full MoveGroup pose-goal plan+execute to
tool_tcp succeeds end-to-end against mock hardware
(demo.launch.py + this parol6_moveit config).

Not yet done: full validation of real_robot.launch.py against a live
bridge/parol6-server end to end (only the individual pieces have been
validated separately so far), and the parol6_moveit vs parol6_bringup
bringup-path duplication (two ways to drive the same hardware interface)
isn't reconciled yet -- both still work independently, not consolidated
into one canonical path.

File: ros_parol/src/parol6_moveit/config/parol6.ros2_control.xacro (robot description, xacro)
@@ -1,10 +1,23 @@
 <?xml version="1.0"?>
 <robot xmlns:xacro="http://www.ros.org/wiki/xacro">
-    <xacro:macro name="parol6_ros2_control" params="name initial_positions_file">
+    <xacro:macro name="parol6_ros2_control"
+                 params="name initial_positions_file use_real_hardware:=false bridge_host:=127.0.0.1 bridge_port:=6001">
         <xacro:property name="initial_positions" value="${load_yaml(initial_positions_file)['initial_positions']}"/>
         <ros2_control name="${name}" type="system">
             <hardware>
-                <!-- By default, set up controllers for simulation. This won't work on real hardware -->
-                <plugin>mock_components/GenericSystem</plugin>
+                <xacro:if value="${use_real_hardware}">
+                    <!-- Talks to a parol6_bridge daemon (TCP loopback), which in turn
+                         talks to parol6-server over UDP using the parol6 Python SDK.
+                         See parol6_hardware_interface and parol6_bridge packages, and
+                         launch/real_robot.launch.py. -->
+                    <plugin>parol6_hardware_interface/Parol6SystemInterface</plugin>
+                    <param name="bridge_host">${bridge_host}</param>
+                    <param name="bridge_port">${bridge_port}</param>
+                    <param name="connect_timeout_sec">10.0</param>
+                </xacro:if>
+                <xacro:unless value="${use_real_hardware}">
+                    <!-- Default: simulation only, no real robot involved. -->
+                    <plugin>mock_components/GenericSystem</plugin>
+                </xacro:unless>
             </hardware>
             <joint name="L1">

File: ros_parol/src/parol6_moveit/config/parol6.urdf.xacro (robot description, xacro)
@@ -1,9 +1,29 @@
 <?xml version="1.0"?>
+<!--
+  tool/tool_variant default to "pneumatic"/"vertical" (not "none") because
+  this MoveIt config plans to the "tool_tcp" frame (see parol6.srdf's
+  arm_group, which now includes tool_tcp_joint as its tip), and tool_tcp's
+  actual position depends on which tool is mounted, see
+  $(find parol6)/urdf/parol6_with_tools.xacro for the full arg
+  documentation. Override at the moveit_config/launch-argument level if a
+  different tool is mounted; every tool variant defines a "tool_tcp_joint"
+  from L6, so the SRDF's chain to it doesn't need to change per tool.
+-->
 <robot xmlns:xacro="http://www.ros.org/wiki/xacro" name="parol6">
     <xacro:arg name="initial_positions_file" default="initial_positions.yaml" />
-    <!-- Import parol6 urdf file -->
-    <xacro:include filename="$(find parol6)/urdf/parol6.urdf" />
+    <xacro:arg name="use_real_hardware" default="false" />
+    <xacro:arg name="bridge_host" default="127.0.0.1" />
+    <xacro:arg name="bridge_port" default="6001" />
+    <xacro:arg name="tool" default="pneumatic" />
+    <xacro:arg name="tool_variant" default="vertical" />
+    <!-- Import parol6 urdf file, with the mounted tool + tool_tcp frame -->
+    <xacro:include filename="$(find parol6)/urdf/parol6_with_tools.xacro" />
     <!-- Import control_xacro -->
     <xacro:include filename="parol6.ros2_control.xacro" />
-    <xacro:parol6_ros2_control name="FakeSystem" initial_positions_file="$(arg initial_positions_file)"/>
+    <xacro:parol6_ros2_control
+        name="FakeSystem"
+        initial_positions_file="$(arg initial_positions_file)"
+        use_real_hardware="$(arg use_real_hardware)"
+        bridge_host="$(arg bridge_host)"
+        bridge_port="$(arg bridge_port)" />
 </robot>
